Commit message: upload urdf

File: CADandURDF/robot_repo/V000_cam/urdf/V000_cam.urdf (robot description, URDF)
Before this commit: robot V000_cam, 14 links, 13 joints
Joints:
- joint body_10: type continuous -> revolute
- joint body_20: type continuous -> revolute
- joint body_30: type continuous -> revolute
