Commit message: vo_model.eval()

File: CADandURDF/robot_repo/broken_feet2/urdf/broken_feet.urdf (robot description, URDF)
Before this commit: robot broken_feet, 14 links, 13 joints
Links:
- link 02: mass 0.141254271685154 -> 0.0831925653721974; geometry collision mesh filename=package://broken_feet/meshes/02.STL; visual mesh filename=package://broken_feet/meshes/02.STL
- link 32: mass 0.0831925653721974 -> 0.141254271685154; geometry collision mesh filename=package://broken_feet/meshes/32.STL; visual mesh filename=package://broken_feet/meshes/32.STL
