Commit message: done

File: CADandURDF/robot_repo/V800_cam/urdf/V800_cam.urdf (robot description, URDF)
Before this commit: robot V800_cam, 14 links, 13 joints
Links:
- link body: mass 1.03 -> 0.727501628669827
Joints:
- joint body_cam: origin xyz=-0.0315000177857023 0.12846719592633 0.0788583994340734 rpy=0.858487020413039 0 0 -> xyz=-0.0315000177857134 0.128467195926324 0.0788583994340782 rpy=-0.712309306 0 0
